File: cad/grip_board/grio_board_test/GR_IO_Board.kicad_pcb (KiCad board)
At the start: 2 copper layers, 99.6 x 44.2 mm, 43 parts, among them J1 Conn_01x04, J2 Conn_01x04, J3 Conn_01x05, J4 Conn_01x05, J5 Conn_01x05, J6 Conn_01x05, J7 Conn_01x04, J8 Conn_01x04, J9 Conn_01x04, SW1 SW_Push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

Commit message: test GR_IO_Board to kicad 6
Other:
- net class Default removed
