File: cad/555-blinker/555-blinker.kicad_pcb (KiCad board)
At the start: 2 copper layers, 59.7 x 36.8 mm, 8 parts, among them U1 LM555

Commit message: migrate to kicad 6
Other:
- net class Default removed

Commit message: attempt to install freeroute plugin in kicad 6
Routing:
- net VCC: track 65.6 -> 55.7 mm
- net Net-(R1-Pad2): track 34.1 -> 27.1 mm
- net GND: track 54.4 -> 49.3 mm
- net Net-(D1-Pad1): track 26.5 -> 23.6 mm
- net Net-(D2-Pad2): track 15.8 -> 14.3 mm, vias 1 -> 0
- net Net-(D1-Pad2): track 22.6 -> 21.2 mm
- net Net-(R2-Pad2): track 12.0 -> 11.4 mm
Changed lines of the file:
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@@
   (gr_line (start 158.75 71.12) (end 99.06 71.12) (layer "Edge.Cuts") (width 0.15))
   (gr_line (start 99.06 71.12) (end 99.06 34.29) (layer "Edge.Cuts") (width 0.15))
-  (segment (start 125.73 43.18) (end 125.73 49.53) (width 0.25) (layer "F.Cu") (net 1))
-  (segment (start 134.62 38.1) (end 134.62 41.91) (width 0.25) (layer "F.Cu") (net 1))
-  (segment (start 127 41.91) (end 125.73 43.18) (width 0.25) (layer "F.Cu") (net 1))
-  (segment (start 104.14 50.8) (end 105.41 49.53) (width 0.25) (layer "F.Cu") (net 1))
-  (segment (start 132.08 53.34) (end 133.35 54.61) (width 0.25) (layer "F.Cu") (net 1))
-  (segment (start 127 53.34) (end 132.08 53.34) (width 0.25) (layer "F.Cu") (net 1))
-  (segment (start 143.51 38.1) (end 134.62 38.1) (width 0.25) (layer "F.Cu") (net 1))
-  (segment (start 125.73 49.53) (end 125.73 52.07) (width 0.25) (layer "F.Cu") (net 1))
-  (segment (start 134.62 41.91) (end 127 41.91) (width 0.25) (layer "F.Cu") (net 1))
-  (segment (start 125.73 52.07) (end 127 53.34) (width 0.25) (layer "F.Cu") (net 1))
-  (segment (start 105.41 49.53) (end 125.73 49.53) (width 0.25) (layer "F.Cu") (net 1))
-  (segment (start 133.35 54.61) (end 133.35 57.15) (width 0.25) (layer "F.Cu") (net 1))
-  (segment (start 104.14 52.07) (end 104.14 50.8) (width 0.25) (layer "F.Cu") (net 1))
-  (segment (start 125.73 57.15) (end 125.73 64.77) (width 0.25) (layer "F.Cu") (net 2))
-  (segment (start 105.41 57.15) (end 104.14 55.88) (width 0.25) (layer "F.Cu") (net 2))
-  (segment (start 127 66.04) (end 148.59 66.04) (width 0.25) (layer "F.Cu") (net 2))
-  (segment (start 125.73 64.77) (end 127 66.04) (width 0.25) (layer "F.Cu") (net 2))
-  (segment (start 104.14 55.88) (end 104.14 54.61) (width 0.25) (layer "F.Cu") (net 2))
-  (segment (start 125.73 57.15) (end 105.41 57.15) (width 0.25) (layer "F.Cu") (net 2))
-  (segment (start 143.51 41.91) (end 143.51 43.18) (width 0.25) (layer "F.Cu") (net 3))
-  (segment (start 139.7 41.91) (end 143.51 41.91) (width 0.25) (layer "F.Cu") (net 3))
-  (segment (start 137.16 41.91) (end 137.16 44.45) (width 0.25) (layer "F.Cu") (net 3))
-  (segment (start 130.81 45.72) (end 130.81 49.53) (width 0.25) (layer "F.Cu") (net 3))
-  (segment (start 132.08 44.45) (end 130.81 45.72) (width 0.25) (layer "F.Cu") (net 3))
-  (segment (start 143.51 43.18) (end 143.51 46.99) (width 0.25) (layer "F.Cu") (net 3))
-  (segment (start 139.7 41.91) (end 137.16 41.91) (width 0.25) (layer "F.Cu") (net 3))
-  (segment (start 137.16 44.45) (end 132.08 44.45) (width 0.25) (layer "F.Cu") (net 3))
-  (segment (start 130.81 54.61) (end 129.54 54.61) (width 0.25) (layer "B.Cu") (net 3))
-  (segment (start 128.27 55.88) (end 128.27 57.15) (width 0.25) (layer "B.Cu") (net 3))
-  (segment (start 129.54 54.61) (end 128.27 55.88) (width 0.25) (layer "B.Cu") (net 3))
-  (segment (start 130.81 49.53) (end 130.81 54.61) (width 0.25) (layer "B.Cu") (net 3))
-  (segment (start 128.27 48.26) (end 128.27 49.53) (width 0.25) (layer "B.Cu") (net 4))
-  (segment (start 138.43 46.99) (end 129.54 46.99) (width 0.25) (layer "B.Cu") (net 4))
-  (segment (start 129.54 46.99) (end 128.27 48.26) (width 0.25) (layer "B.Cu") (net 4))
-  (segment (start 147.32 43.18) (end 147.32 55.88) (width 0.25) (layer "F.Cu") (net 5))
-  (segment (start 147.32 55.88) (end 144.78 55.88) (width 0.25) (layer "F.Cu") (net 5))
-  (segment (start 144.78 55.88) (end 143.51 57.15) (width 0.25) (layer "F.Cu") (net 5))
-  (segment (start 148.59 41.91) (end 147.32 43.18) (width 0.25) (layer "F.Cu") (net 5))
-  (segment (start 148.59 38.1) (end 148.59 41.91) (width 0.25) (layer "F.Cu") (net 5))
-  (segment (start 154.94 59.69) (end 154.94 59.69) (width 0.25) (layer "F.Cu") (net 6))
-  (segment (start 154.94 53.34) (end 154.94 59.69) (width 0.25) (layer "F.Cu") (net 6))
-  (via (at 154.94 59.69) (size 0.8) (drill 0.4) (layers "F.Cu" "B.Cu") (net 6))
-  (segment (start 152.4 59.69) (end 151.13 60.96) (width 0.25) (layer "B.Cu") (net 6))
-  (segment (start 151.13 60.96) (end 151.13 66.04) (width 0.25) (layer "B.Cu") (net 6))
-  (segment (start 154.94 59.69) (end 152.4 59.69) (width 0.25) (layer "B.Cu") (net 6))
-  (segment (start 149.86 53.34) (end 149.86 58.42) (width 0.25) (layer "F.Cu") (net 7))
-  (segment (start 132.08 59.69) (end 130.81 58.42) (width 0.25) (layer "F.Cu") (net 7))
-  (segment (start 130.81 58.42) (end 130.81 57.15) (width 0.25) (layer "F.Cu") (net 7))
-  (segment (start 149.86 58.42) (end 148.59 59.69) (width 0.25) (layer "F.Cu") (net 7))
-  (segment (start 148.59 59.69) (end 143.51 59.69) (width 0.25) (layer "F.Cu") (net 7))
-  (segment (start 143.51 59.69) (end 132.08 59.69) (width 0.25) (layer "F.Cu") (net 7))
+  (segment (start 107.8553 49.53) (end 125.73 49.53) (width 0.25) (layer "F.Cu") (net 1))
+  (segment (start 104.14 52.07) (end 105.3153 52.07) (width 0.25) (layer "F.Cu") (net 1))
+  (segment (start 138.43 38.1) (end 134.62 41.91) (width 0.25) (layer "F.Cu") (net 1))
+  (segment (start 105.3153 52.07) (end 107.8553 49.53) (width 0.25) (layer "F.Cu") (net 1))
+  (segment (start 143.51 38.1) (end 138.43 38.1) (width 0.25) (layer "F.Cu") (net 1))
+  (segment (start 133.35 57.15) (end 133.35 56.0247) (width 0.25) (layer "B.Cu") (net 1))
+  (segment (start 126.3282 49.5655) (end 126.6094 49.5655) (width 0.25) (layer "B.Cu") (net 1))
+  (segment (start 133.0687 56.0247) (end 133.35 56.0247) (width 0.25) (layer "B.Cu") (net 1))
+  (segment (start 126.6094 49.5655) (end 126.6095 49.5654) (width 0.25) (layer "B.Cu") (net 1))
+  (segment (start 126.6095 49.5654) (end 134.2649 41.91) (width 0.25) (layer "B.Cu") (net 1))
+  (segment (start 125.73 49.53) (end 126.2927 49.53) (width 0.25) (layer "B.Cu") (net 1))
+  (segment (start 126.6095 49.5654) (end 133.0687 56.0247) (width 0.25) (layer "B.Cu") (net 1))
+  (segment (start 134.2649 41.91) (end 134.62 41.91) (width 0.25) (layer "B.Cu") (net 1))
+  (segment (start 126.2927 49.53) (end 126.3282 49.5655) (width 0.25) (layer "B.Cu") (net 1))
+  (segment (start 125.73 57.15) (end 124.6047 57.15) (width 0.25) (layer "F.Cu") (net 2))
+  (segment (start 135.464 66.04) (end 126.8553 57.4313) (width 0.25) (layer "F.Cu") (net 2))
+  (segment (start 126.8553 57.4313) (end 126.8553 57.15) (width 0.25) (layer "F.Cu") (net 2))
+  (segment (start 104.14 54.61) (end 122.0647 54.61) (width 0.25) (layer "F.Cu") (net 2))
+  (segment (start 125.73 57.15) (end 126.8553 57.15) (width 0.25) (layer "F.Cu") (net 2))
+  (segment (start 122.0647 54.61) (end 124.6047 57.15) (width 0.25) (layer "F.Cu") (net 2))
+  (segment (start 148.59 66.04) (end 135.464 66.04) (width 0.25) (layer "F.Cu") (net 2))
+  (segment (start 130.81 53.4847) (end 130.81 49.53) (width 0.25) (layer "F.Cu") (net 3))
+  (segment (start 128.27 56.0247) (end 130.81 53.4847) (width 0.25) (layer "F.Cu") (net 3))
+  (segment (start 128.27 57.15) (end 128.27 56.0247) (width 0.25) (layer "F.Cu") (net 3))
+  (segment (start 130.81 49.53) (end 131.9353 49.53) (width 0.25) (layer "B.Cu") (net 3))
+  (segment (start 138.2487 42.9353) (end 139.7 42.9353) (width 0.25) (layer "B.Cu") (net 3))
+  (segment (start 143.51 46.7453) (end 139.7 42.9353) (width 0.25) (layer "B.Cu") (net 3))
+  (segment (start 139.7 41.91) (end 139.7 42.9353) (width 0.25) (layer "B.Cu") (net 3))
+  (segment (start 143.51 46.99) (end 143.51 46.7453) (width 0.25) (layer "B.Cu") (net 3))
+  (segment (start 131.9353 49.53) (end 131.9353 49.2487) (width 0.25) (layer "B.Cu") (net 3))
+  (segment (start 131.9353 49.2487) (end 138.2487 42.9353) (width 0.25) (layer "B.Cu") (net 3))
+  (segment (start 129.3953 49.53) (end 129.3953 49.2487) (width 0.25) (layer "F.Cu") (net 4))
+  (segment (start 129.3953 49.2487) (end 131.654 46.99) (width 0.25) (layer "F.Cu") (net 4))
+  (segment (start 128.27 49.53) (end 129.3953 49.53) (width 0.25) (layer "F.Cu") (net 4))
+  (segment (start 131.654 46.99) (end 138.43 46.99) (width 0.25) (layer "F.Cu") (net 4))
+  (segment (start 148.59 52.07) (end 143.51 57.15) (width 0.25) (layer "B.Cu") (net 5))
+  (segment (start 148.59 38.1) (end 148.59 52.07) (width 0.25) (layer "B.Cu") (net 5))
+  (segment (start 154.94 62.23) (end 154.94 53.34) (width 0.25) (layer "B.Cu") (net 6))
+  (segment (start 151.13 66.04) (end 154.94 62.23) (width 0.25) (layer "B.Cu") (net 6))
+  (segment (start 131.9353 57.4313) (end 134.194 59.69) (width 0.25) (layer "F.Cu") (net 7))
+  (segment (start 130.81 57.15) (end 131.9353 57.15) (width 0.25) (layer "F.Cu") (net 7))
+  (segment (start 134.194 59.69) (end 143.51 59.69) (width 0.25) (layer "F.Cu") (net 7))
+  (segment (start 131.9353 57.15) (end 131.9353 57.4313) (width 0.25) (layer "F.Cu") (net 7))
+  (segment (start 143.51 58.4647) (end 144.7353 58.4647) (width 0.25) (layer "B.Cu") (net 7))
+  (segment (start 143.51 59.69) (end 143.51 58.4647) (width 0.25) (layer "B.Cu") (net 7))
+  (segment (start 144.7353 58.4647) (end 149.86 53.34) (width 0.25) (layer "B.Cu") (net 7))
 )
