File: cad/5LED-TH/5LED-TH.kicad_pcb (KiCad board)
At the start: 2 copper layers, 40.6 x 30.5 mm, 11 parts, among them J1 Screw_Terminal_01x02

Commit message: added mounting holes
Parts:
- added REF**: MountingHole_3.2mm_M3_DIN965_Pad, MountingHole:MountingHole_3.2mm_M3_DIN965_Pad, F.Cu at (38.0, 18.0)
- added REF**: MountingHole_3.2mm_M3_DIN965_Pad, MountingHole:MountingHole_3.2mm_M3_DIN965_Pad, F.Cu at (37.0, 38.0)
Routing:
- net GND: track 48.7 -> 60.0 mm
Other:
- outline, holes or cut-outs redrawn
Changed lines of the file:
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@@
     )
+  )
+  (footprint "MountingHole:MountingHole_3.2mm_M3_DIN965_Pad" (layer "F.Cu")
+    (at 38 18)
+    (descr "Mounting Hole 3.2mm, M3, DIN965")
+    (tags "mounting hole 3.2mm m3 din965")
+    (attr exclude_from_pos_files exclude_from_bom)
+    (fp_text reference "REF**" (at 0 -3.8) (layer "F.SilkS")
+      (effects (font (size 1 1) (thickness 0.15)))
+    )
+    (fp_text value "MountingHole_3.2mm_M3_DIN965_Pad" (at 0 3.8) (layer "F.Fab")
+      (effects (font (size 1 1) (thickness 0.15)))
+    )
+    (fp_text user "${REFERENCE}" (at 0 0) (layer "F.Fab")
+      (effects (font (size 1 1) (thickness 0.15)))
+    )
+    (fp_circle (center 0 0) (end 2.8 0) (layer "Cmts.User") (width 0.15) (fill none))
+    (fp_circle (center 0 0) (end 3.05 0) (layer "F.CrtYd") (width 0.05) (fill none))
+    (pad "1" thru_hole circle (at 0 0) (size 5.6 5.6) (drill 3.2) (layers *.Cu *.Mask)
+      (net 1 "GND"))
   )
   (footprint "Resistor_THT:R_Axial_DIN0204_L3.6mm_D1.6mm_P5.08mm_Horizontal" (layer "F.Cu")
@@
       (rotate (xyz 0 0 0))
     )
+  )
+  (footprint "MountingHole:MountingHole_3.2mm_M3_DIN965_Pad" (layer "F.Cu")
+    (at 37 38)
+    (descr "Mounting Hole 3.2mm, M3, DIN965")
+    (tags "mounting hole 3.2mm m3 din965")
+    (attr exclude_from_pos_files exclude_from_bom)
+    (fp_text reference "REF**" (at 0 -3.8) (layer "F.SilkS")
+      (effects (font (size 1 1) (thickness 0.15)))
+    )
+    (fp_text value "MountingHole_3.2mm_M3_DIN965_Pad" (at 0 3.8) (layer "F.Fab")
+      (effects (font (size 1 1) (thickness 0.15)))
+    )
+    (fp_text user "${REFERENCE}" (at 0 0) (layer "F.Fab")
+      (effects (font (size 1 1) (thickness 0.15)))
+    )
+    (fp_circle (center 0 0) (end 2.8 0) (layer "Cmts.User") (width 0.15) (fill none))
+    (fp_circle (center 0 0) (end 3.05 0) (layer "F.CrtYd") (width 0.05) (fill none))
+    (pad "1" thru_hole circle (at 0 0) (size 5.6 5.6) (drill 3.2) (layers *.Cu *.Mask))
   )
   (footprint "Resistor_THT:R_Axial_DIN0204_L3.6mm_D1.6mm_P5.08mm_Horizontal" (layer "F.Cu")
@@
       (xy 66.548 13.208)
     ) (layer "Edge.Cuts") (width 0.15) (fill none))
+  (gr_circle (center 31 40) (end 31 41) (layer "Edge.Cuts") (width 0.15) (fill none))
+  (gr_circle (center 31 16) (end 31 17) (layer "Edge.Cuts") (width 0.15) (fill none))
+  (segment (start 38 18) (end 35 18) (width 0.1524) (layer "F.Cu") (net 1))
+  (segment (start 34.036 19.036) (end 34.036 25.908) (width 0.1524) (layer "F.Cu") (net 1))
   (segment (start 55.29 25.908) (end 34.036 25.908) (width 0.1524) (layer "F.Cu") (net 1))
   (segment (start 57.7991 28.6993) (end 57.7991 28.4171) (width 0.1524) (layer "F.Cu") (net 1))
@@
   (segment (start 57.7991 28.4171) (end 55.6472 26.2651) (width 0.1524) (layer "F.Cu") (net 1))
   (segment (start 58.928 28.6993) (end 57.7991 28.6993) (width 0.1524) (layer "F.Cu") (net 1))
+  (segment (start 34 19) (end 34.036 19.036) (width 0.1524) (layer "F.Cu") (net 1))
+  (segment (start 35 18) (end 34 19) (width 0.1524) (layer "F.Cu") (net 1))
   (segment (start 58.928 28.6993) (end 58.928 34.4143) (width 0.1524) (layer "B.Cu") (net 1))
   (segment (start 58.928 17.2693) (end 58.928 22.9843) (width 0.1524) (layer "B.Cu") (net 1))
