File: cad/555-flasher/555 Timer LED Flasher.kicad_pcb (KiCad board)
At the start: 2 copper layers, 61 x 25.4 mm, 8 parts, among them U1 NE555D

Commit message: added switch box
Other:
- net class Default removed
